File: light/kicad/light.kicad_sch (KiCad schematic)
At the start: 106 parts, among them J1 Conn_01x03_Pin, J2 Conn_01x02_Pin, J3 SPI Socket, U1 FT4232H, U11 TLV7103318DDSE, U14 74LVC1G07, U2 SN74AVC4T774RSVR, U3 SN74AVC4T774RSVR, U4 SN74AVC4T774RSVR, U5 74LVC1G07, U6 SN74AHC595QWBQBRQ1, U7 TLV75533PDBV, U8 TLV75533PDBV, U9 93LC56BT-I/OT, Y1 12MHz_7M-12.000MAAJ

Commit message: kicad: add footprints and upload new placement
1. change JDB11 package footprint
2.  add footrprint for J3
3.  Change U6 footprint to WQFN
Parts:
- J1: footprint (none) -> Connector_PinHeader_2.54mm:PinHeader_1x03_P2.54mm_Vertical
- J2: footprint Connector_PinHeader_2.54mm:PinHeader_1x02_P2.54mm_Vertical_SMD_Pin1Left -> Connector_PinHeader_2.54mm:PinHeader_1x02_P2.54mm_Vertical
- J3: footprint ACES_50950-0084N-002 -> (none)
- JDB11: footprint Connector_PinHeader_1.27mm:PinHeader_2x05_P1.27mm_Vertical_SMD -> (none)
- JECDB1: footprint HRS_FH19C-10S-0.5SH -> (none)
- LED2, LED7: footprint EAST1616RGBA1 -> (none)
- U14, U5: footprint Library_Myself:SOT-23-5_L3.0-W1.7-P0.95-LS2.8-BR -> Package_SON:Texas_X2SON-5_0.8x0.8mm_P0.48mm_RoutingVia
- U6: footprint Library_Myself:TSSOP-16_L5.0-W4.4-P0.65-LS6.4-BL -> 0JLC:DHVQFN-16_L3.5-W2.5-P0.50-BL-EP
Changed lines of the file:
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@@
 			)
 		)
-		(property "Footprint" "Library_Myself:TSSOP-16_L5.0-W4.4-P0.65-LS6.4-BL"
+		(property "Footprint" "0JLC:DHVQFN-16_L3.5-W2.5-P0.50-BL-EP"
 			(at 74.93 254 0)
 			(effects
@@
 			)
 		)
-		(property "Footprint" "EAST1616RGBA1"
+		(property "Footprint" ""
 			(at 137.16 266.7 0)
 			(effects
@@
 			)
 		)
-		(property "Footprint" "Library_Myself:SOT-23-5_L3.0-W1.7-P0.95-LS2.8-BR"
+		(property "Footprint" "Package_SON:Texas_X2SON-5_0.8x0.8mm_P0.48mm_RoutingVia"
 			(at 264.16 184.15 0)
 			(effects
@@
 			)
 		)
-		(property "Footprint" ""
+		(property "Footprint" "Connector_PinHeader_2.54mm:PinHeader_1x03_P2.54mm_Vertical"
 			(at 146.05 24.13 0)
 			(effects
@@
 			)
 		)
-		(property "Footprint" "Library_Myself:SOT-23-5_L3.0-W1.7-P0.95-LS2.8-BR"
+		(property "Footprint" "Package_SON:Texas_X2SON-5_0.8x0.8mm_P0.48mm_RoutingVia"
 			(at 283.21 208.28 0)
 			(effects
@@
 			)
 		)
-		(property "Footprint" "EAST1616RGBA1"
+		(property "Footprint" ""
 			(at 52.07 226.06 0)
 			(effects
@@
 			)
 		)
-		(property "Footprint" "ACES_50950-0084N-002"
+		(property "Footprint" ""
 			(at 339.09 55.88 0)
 			(effects
@@
 			)
 		)
-		(property "Footprint" "Connector_PinHeader_1.27mm:PinHeader_2x05_P1.27mm_Vertical_SMD"
+		(property "Footprint" ""
 			(at 326.39 96.52 0)
 			(effects
@@
 			)
 		)
-		(property "Footprint" "Connector_PinHeader_2.54mm:PinHeader_1x02_P2.54mm_Vertical_SMD_Pin1Left"
+		(property "Footprint" "Connector_PinHeader_2.54mm:PinHeader_1x02_P2.54mm_Vertical"
 			(at 367.03 17.78 0)
 			(effects
@@
 			)
 		)
-		(property "Footprint" "HRS_FH19C-10S-0.5SH"
+		(property "Footprint" ""
 			(at 393.7 17.78 0)
 			(effects
